File: kicad/rosalyn-rx.kicad_pcb (KiCad board)
At the start: 4 copper layers, 35 x 20.6 mm, 36 parts, among them J2 Serial1, J3 Serial2, J4 PWM, U1 STM32F303CCTx, U2 E22-EBYTE, U3 XC6206P330MR, U4 TXS0108EPW, U5 BMP280, U6 ICM-20602

Commit message: updated nvdata driver
Connections:
- net e22_busy renamed radio_busy
- net e22_dio1 renamed radio_dio1
- net e22_dio2 renamed radio_dio2
- net e22_nrst renamed radio_nrst
- net e22_nss renamed radio_nss
- net e22_rxen renamed radio_rxen
- net e22_txen renamed radio_txen
